Commit message: primary changes

File: urdf/base.urdf (robot description, URDF)
Before this commit: robot base, 4 links, 3 joints
Links:
- link base_link: geometry collision mesh filename=/home/alwin/catkin_ws/src/base/meshes/base_link.STL; visual mesh filename=/home/alwin/catkin_ws/src/base/meshes/base_link.STL
- link wheel_1: geometry collision mesh filename=/home/alwin/catkin_ws/src/base/meshes/wheel_1.STL; visual mesh filename=/home/alwin/catkin_ws/src/base/meshes/wheel_1.STL
- link wheel_2: geometry collision mesh filename=/home/alwin/catkin_ws/src/base/meshes/wheel_1.STL; visual mesh filename=/home/alwin/catkin_ws/src/base/meshes/wheel_1.STL
- link wheel_3: geometry collision mesh filename=/home/alwin/catkin_ws/src/base/meshes/wheel_1.STL; visual mesh filename=/home/alwin/catkin_ws/src/base/meshes/wheel_1.STL
Joints:
- joint revolute_1: type revolute -> continuous
- joint revolute_2: type revolute -> continuous
- joint revolute_3: type revolute -> continuous
